Commit message: lidar urdf added

File: bb_description/urdf/bb.urdf.xacro (robot description, xacro)
@@ -136,5 +136,5 @@
       <origin xyz="3.8996812895542E-07 2.40073004698083E-07 0.00219173397061509" rpy="0 0 0" />
       <mass value="1.44379265037902E-06" />
-      <inertia ixx="7.23075276010246E-11" ixy="-6.10956872363424E-16" ixz="2.22849693527207E-15"
+      <inertia ixx="7.23075276010246E-11" ixy="-6.10956872363424E-16" ixz="2.22849693525031E-15"
                iyy="3.87137930859167E-11" iyz="2.939098587861E-15"
                izz="1.00967486676306E-10" />
@@ -172,4 +172,7 @@
         <mesh filename="package://bb_description/meshes/imu_link.STL" />
       </geometry>
+      <material name="imu_blue">
+        <color rgba="0.2 0.4 0.8 1.0"/>
+      </material>
     </visual>
     <collision>
@@ -184,4 +187,35 @@
     <parent link="base_link" />
     <child link="imu_link" />
+    <axis xyz="0 0 0" />
+  </joint>
+  <!-- LIDAR Link and Joint -->
+  <link name="lidar_link">
+    <inertial>
+      <origin xyz="-0.0001282412 0.0054365480 0.0157879479" rpy="0 0 0"/>
+      <mass value="0.1700000000"/>
+      <inertia ixx="1.3580113591e-04" ixy="3.5050643277e-08" ixz="-3.2031016417e-07"
+               iyy="1.4486144937e-04" iyz="-1.3760036381e-05"
+               izz="2.2843409170e-05" />
+    </inertial>
+    <visual>
+      <origin xyz="0 0 0" rpy="0 0 0" />
+      <geometry>
+        <cylinder radius="0.022" length="0.026"/>
+      </geometry>
+      <material name="lidar_blue">
+        <color rgba="0.2 0.4 0.8 1.0"/>
+      </material>
+    </visual>
+    <collision>
+      <origin xyz="0 0 0" rpy="0 0 0" />
+      <geometry>
+        <cylinder radius="0.022" length="0.026"/>
+      </geometry>
+    </collision>
+  </link>
+  <joint name="lidar_joint" type="fixed">
+    <origin xyz="0 0 0.084" rpy="0 0 0" />
+    <parent link="base_link" />
+    <child link="lidar_link" />
     <axis xyz="0 0 0" />
   </joint>

Commit message: lidar weight adjusted

File: bb_description/urdf/bb.urdf.xacro (robot description, xacro)
@@ -193,8 +193,8 @@
     <inertial>
       <origin xyz="-0.0001282412 0.0054365480 0.0157879479" rpy="0 0 0"/>
-      <mass value="0.1700000000"/>
-      <inertia ixx="1.3580113591e-04" ixy="3.5050643277e-08" ixz="-3.2031016417e-07"
-               iyy="1.4486144937e-04" iyz="-1.3760036381e-05"
-               izz="2.2843409170e-05" />
+      <mass value="0.0600000000"/>
+      <inertia ixx="4.80e-05" ixy="1.24e-08" ixz="-1.13e-07"
+          iyy="5.11e-05" iyz="-4.86e-06"
+          izz="8.07e-06"/>
     </inertial>
     <visual>
